Commit message: update

File: assets/hab_stretch/urdf/stretch.urdf (robot description, URDF)
Before this commit: robot stretch_description, 44 links, 43 joints
Links:
- removed link link_straight_gripper
- added link base_imu, mass 0.00092; collision mesh filename=package://stretch_description/meshes/base_imu.STL; visual mesh filename=package://stretch_description/meshes/base_imu.STL
- added link link_aruco_d405, mass 0.000393662237156561; collision mesh filename=package://stretch_description/meshes/link_SG3_aruco_d405.STL; visual mesh filename=package://stretch_description/meshes/link_SG3_aruco_d405.STL
- added link link_aruco_fingertip_left, mass 7.44175884388882e-05; collision mesh filename=package://stretch_description/meshes/link_SG3_aruco_fingert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; visual mesh filename=package://stretch_description/meshes/link_SG3_aruco_fingert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
- added link link_aruco_fingertip_right, mass 7.44175884388862e-05; collision mesh filename=package://stretch_description/meshes/link_SG3_aruco_fingert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; visual mesh filename=package://stretch_description/meshes/link_SG3_aruco_fingert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
- added link link_grasp_center
- added link link_gripper_s3_body, mass 0.288995995074102; collision mesh filename=package://stretch_description/meshes/link_SG3_gripper_body_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; visual mesh filename=package://stretch_description/meshes/link_SG3_gripper_body.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
- added link link_head_nav_cam, mass 0.028346169831483; collision mesh filename=package://stretch_description/meshes/link_SE3_head_nav_cam_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; visual mesh filename=package://stretch_description/meshes/link_SE3_head_nav_cam.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
- added link link_wrist_quick_connect
- link base_link: mass 1.0723782659782 -> 17.384389; geometry collision mesh filename=package://stretch_description/meshes/base_link_collision.STL; visual mesh filename=package://stretch_description/meshes/base_link.STL
- link camera_link: geometry collision box size=0.02505 0.09 0.025; visual mesh filename=package://stretch_description/meshes/d435.dae
- link caster_link: geometry collision sphere radius=0.032; visual mesh filename=package://stretch_description/meshes/omni_wheel_m.STL
- link laser: mass 0.0749979022894495 -> 0.216007; geometry collision mesh filename=package://stretch_description/meshes/laser_collision.STL; visual mesh filename=package://stretch_description/meshes/laser.STL
- link link_arm_l0: mass 0.101241250325294 -> 0.427734; geometry collision mesh filename=package://stretch_description/meshes/link_arm_l0_collision.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; visual mesh filename=package://stretch_description/meshes/link_arm_l0.STL
- link link_arm_l1: mass 0.0511763619538321 -> 0.113658; geometry collision mesh filename=package://stretch_description/meshes/link_arm_l1_collision.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; visual mesh filename=package://stretch_description/meshes/link_arm_l1.STL
- link link_arm_l2: mass 0.0569074368576238 -> 0.130565; geometry collision mesh filename=package://stretch_description/meshes/link_arm_l2_collision.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; visual mesh filename=package://stretch_description/meshes/link_arm_l2.STL
- link link_arm_l3: mass 0.0626921047058405 -> 0.146817; geometry collision mesh filename=package://stretch_description/meshes/link_arm_l3_collision.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; visual mesh filename=package://stretch_description/meshes/link_arm_l3.STL
- link link_arm_l4: mass 0.0676525455789735 -> 0.235626; geometry collision mesh filename=package://stretch_description/meshes/link_arm_l4_collision.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; visual mesh filename=package://stretch_description/meshes/link_arm_l4.STL
- link link_aruco_inner_wrist: mass 0 -> 0.0; geometry collision mesh filename=package://stretch_description/meshes/link_aruco_inner_wrist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; visual mesh filename=package://stretch_description/meshes/link_aruco_inner_wrist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
- link link_aruco_left_base: mass 3.59999999990368E-06 -> 3.59999999990368e-06; geometry collision mesh filename=package://stretch_description/meshes/link_aruco_left_base.S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; visual mesh filename=package://stretch_description/meshes/link_aruco_left_base.S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
- link link_aruco_right_base: mass 3.59999999990368E-06 -> 3.59999999990368e-06; geometry collision mesh filename=package://stretch_description/meshes/link_aruco_right_base.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; visual mesh filename=package://stretch_description/meshes/link_aruco_right_base.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
- link link_aruco_shoulder: mass 0 -> 0.0; geometry collision mesh filename=package://stretch_description/meshes/link_aruco_shoulder.STL; visual mesh filename=package://stretch_description/meshes/link_aruco_shoulder.STL
- link link_aruco_top_wrist: mass 0 -> 0.0; geometry collision mesh filename=package://stretch_description/meshes/link_aruco_top_wrist.S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; visual mesh filename=package://stretch_description/meshes/link_aruco_top_wrist.S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
- link link_gripper_finger_left: mass 0.0476207785199479 -> 0.0483698266031602; geometry collision mesh filename=package://stretch_description/meshes/link_SG3_gripper_finge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; visual mesh filename=package://stretch_description/meshes/link_SG3_gripper_finge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
- link link_gripper_finger_right: mass 0.047621 -> 0.0483698337858479; geometry collision mesh filename=package://stretch_description/meshes/link_SG3_gripper_finge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; visual mesh filename=package://stretch_description/meshes/link_SG3_gripper_finge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
- link link_gripper_fingertip_left: mass 0.00382160686584851 -> 0.00382162054362131; geometry collision mesh filename=package://stretch_description/meshes/link_SG3_gripper_finge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; visual mesh filename=package://stretch_description/meshes/link_SG3_gripper_finge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
- link link_gripper_fingertip_right: mass 0.00382160881468841 -> 0.00382162062525088; geometry collision mesh filename=package://stretch_description/meshes/link_SG3_gripper_finge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; visual mesh filename=package://stretch_description/meshes/link_SG3_gripper_finge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
- link link_head: mass 0.129454717596498 -> 0.681871; geometry collision mesh filename=package://stretch_description/meshes/link_head_collision.STL; visual mesh filename=package://stretch_description/meshes/link_head.STL
- link link_head_pan: mass 0.035858341182617 -> 0.062462; geometry collision mesh filename=package://stretch_description/meshes/link_head_pan_collisio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; visual mesh filename=package://stretch_description/meshes/link_head_pan.STL
- link link_head_tilt: mass 0.0701242408063442 -> 0.283548; geometry collision mesh filename=package://stretch_description/meshes/link_head_tilt_collisi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; visual mesh filename=package://stretch_description/meshes/link_head_tilt.STL
- link link_left_wheel: mass 0.01 -> 0.20773; geometry collision mesh filename=package://stretch_description/meshes/link_left_wheel_collis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; visual mesh filename=package://stretch_description/meshes/link_left_wheel.STL
- link link_lift: mass 0.444820831236007 -> 1.987167; geometry collision mesh filename=package://stretch_description/meshes/link_lift_collision.STL; visual mesh filename=package://stretch_description/meshes/link_lift.STL
- link link_mast: mass 0.749143203376401 -> 1.764017; geometry collision mesh filename=package://stretch_description/meshes/link_mast_collision.STL; visual mesh filename=package://stretch_description/meshes/link_mast.STL
- link link_right_wheel: mass 0.01 -> 0.20773; geometry collision mesh filename=package://stretch_description/meshes/link_right_wheel_colli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; visual mesh filename=package://stretch_description/meshes/link_right_wheel.STL
- link link_wrist_pitch: mass 0.0701267146295583 -> 0.116590512374845; geometry collision mesh filename=package://stretch_description/meshes/link_DW3_wrist_pitch_c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; visual mesh filename=package://stretch_description/meshes/link_DW3_wrist_pitch.S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
- link link_wrist_roll: mass 0.00585666394358811 -> 0.0221916689638078; geometry collision mesh filename=package://stretch_description/meshes/link_DW3_wrist_roll_co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; visual mesh filename=package://stretch_description/meshes/link_DW3_wrist_roll.STL
- link link_wrist_yaw: mass 0.0405398981326229 -> 0.054422; geometry collision mesh filename=package://stretch_description/meshes/link_wrist_yaw_collisi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; visual mesh filename=package://stretch_description/meshes/link_wrist_yaw.STL
- link link_wrist_yaw_bottom: mass 0.0988906816399982 -> 0.144548635554334; geometry collision mesh filename=package://stretch_description/meshes/link_DW3_wrist_yaw_bot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; visual mesh filename=package://stretch_description/meshes/link_DW3_wrist_yaw_bot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
- link respeaker_base: mass 0.00969129410417277 -> 0.025175; geometry collision mesh filename=package://stretch_description/meshes/respeaker_base.STL; visual mesh filename=package://stretch_description/meshes/respeaker_base.STL
Joints:
- removed joint joint_straight_gripper
- added joint joint_aruco_d405: type fixed, parent link_gripper_s3_body, child link_aruco_d405, origin xyz=0.0 0.0671264013906604 0.0297716109784749 rpy=2.96705999342568 -0.000305721573415565 3.1398588194619, axis 0.0 0.0 0.0
- added joint joint_aruco_fingertip_left: type fixed, parent link_gripper_finger_left, child link_aruco_fingertip_left, origin xyz=0.143934974292929 -0.00436381846064454 -8.58640479230455e-05 rpy=-1.76278254451424 0.0 0.959931088596885, axis 0.0 0.0 0.0
- added joint joint_aruco_fingertip_right: type fixed, parent link_gripper_finger_right, child link_aruco_fingertip_right, origin xyz=-0.143934974292953 -0.00436381846065068 -8.58640479174944e-05 rpy=-1.76278254451426 0.0 -0.959931088596862, axis 0.0 0.0 0.0
- added joint joint_base_imu: type fixed, parent base_link, child base_imu, origin xyz=-0.12838 0.0031592 0.1474 rpy=-3.1416 0.0 -1.5708, axis 0.0 0.0 0.0
- added joint joint_grasp_center: type fixed, parent link_gripper_s3_body, child link_grasp_center, origin xyz=0.0 0.0 0.23 rpy=-1.5707963267949 -1.5707963267948 0.0
- added joint joint_gripper_s3_body: type fixed, parent link_wrist_roll, child link_gripper_s3_body, origin xyz=0.0 0.0 0.0209999999993159 rpy=0.0 0.0 -3.14159265358975, axis 0.0 0.0 0.0
- added joint joint_head_nav_cam: type fixed, parent link_head_tilt, child link_head_nav_cam, origin xyz=0.0402000000000069 -0.0411729746231231 -0.0245785717313561 rpy=0.0 1.5707963267949 0.0, axis 0.0 0.0 0.0
- added joint joint_wrist_quick_connect: type fixed, parent link_wrist_roll, child link_wrist_quick_connect, origin xyz=0.0 0.0 0.0085 rpy=1.5708 0.0 -1.5708, axis 0.0 0.0 0.0
- joint camera_accel_joint: origin xyz=-0.01174 -0.00552 0.0051 rpy=0 0 0 -> xyz=-0.01174 -0.00552 0.0051 rpy=0.0 0.0 0.0
- joint camera_accel_optical_joint: origin xyz=0 0 0 rpy=-1.5707963267948966 0 -1.5707963267948966 -> xyz=0.0 0.0 0.0 rpy=-1.5707963267948966 0.0 -1.5707963267948966
- joint camera_color_joint: origin xyz=0 0.015 0 rpy=0 0 0 -> xyz=0.0 0.015 0.0 rpy=0.0 0.0 0.0
- joint camera_color_optical_joint: origin xyz=0 0 0 rpy=-1.5707963267948966 0 -1.5707963267948966 -> xyz=0.0 0.0 0.0 rpy=-1.5707963267948966 0.0 -1.5707963267948966
- joint camera_depth_joint: origin xyz=0 0 0 rpy=0 0 0 -> xyz=0.0 0.0 0.0 rpy=0.0 0.0 0.0
- joint camera_depth_optical_joint: origin xyz=0 0 0 rpy=-1.5707963267948966 0 -1.5707963267948966 -> xyz=0.0 0.0 0.0 rpy=-1.5707963267948966 0.0 -1.5707963267948966
- joint camera_gyro_joint: origin xyz=-0.01174 -0.00552 0.0051 rpy=0 0 0 -> xyz=-0.01174 -0.00552 0.0051 rpy=0.0 0.0 0.0
- joint camera_gyro_optical_joint: origin xyz=0 0 0 rpy=-1.5707963267948966 0 -1.5707963267948966 -> xyz=0.0 0.0 0.0 rpy=-1.5707963267948966 0.0 -1.5707963267948966
- joint camera_infra1_joint: origin xyz=0 0.0 0 rpy=0 0 0 -> xyz=0.0 0.0 0.0 rpy=0.0 0.0 0.0
- joint camera_infra1_optical_joint: origin xyz=0 0 0 rpy=-1.5707963267948966 0 -1.5707963267948966 -> xyz=0.0 0.0 0.0 rpy=-1.5707963267948966 0.0 -1.5707963267948966
- joint camera_infra2_joint: origin xyz=0 -0.05 0 rpy=0 0 0 -> xyz=0.0 -0.05 0.0 rpy=0.0 0.0 0.0
- joint camera_infra2_optical_joint: origin xyz=0 0 0 rpy=-1.5707963267948966 0 -1.5707963267948966 -> xyz=0.0 0.0 0.0 rpy=-1.5707963267948966 0.0 -1.5707963267948966
- joint camera_joint: origin xyz=0.03 -0.0122 0.0182 rpy=0.0 0.0 0.0 -> xyz=0.026655671416476928 -0.008521482915378683 0.018242446870766118 rpy=0.004952633977773744 0.0006938647732388503 -0.08642937619799977
- joint camera_link_joint: origin xyz=0.010600000000000002 0.0175 0.0125 rpy=0 0 0 -> xyz=0.010600000000000002 0.0175 0.0125 rpy=0.0 0.0 0.0
- joint caster_joint: axis 0 0 1 -> 0.0 0.0 1.0; origin xyz=-0.245 0.0 0.032 rpy=-1.5707963267948966 0 0 -> xyz=-0.245 0.0 0.032 rpy=-1.5707963267948966 0.0 0.0
- joint joint_arm_l0: axis 0 0 1 -> 0.0 0.0 1.0; limit lower=0.0 upper=0.13 effort=100 velocity=1.0 -> lower=0.0 upper=0.13 effort=100.0 velocity=1.0; origin xyz=0 0 -0.0137499999999938 rpy=-3.05317390622457E-16 -4.23236224076729E-16 -2.68425135229209E-17 -> xyz=0.0 0.0 -0.0137499999991968 rpy=7.63746778746202e-30 -3.80121128864402e-15 2.62707547767438e-15
- joint joint_arm_l1: axis 0 0 1 -> 0.0 0.0 1.0; limit lower=0.0 upper=0.13 effort=100 velocity=1.0 -> lower=0.0 upper=0.13 effort=100.0 velocity=1.0; origin xyz=0 0 0.013 rpy=7.41596560408007E-17 1.33876788296791E-16 -2.44545873596083E-16 -> xyz=0.0 0.0 0.0129999999999981 rpy=-7.63746778746202e-30 -7.88860905221012e-31 1.11022302462516e-16
- joint joint_arm_l2: axis 0 0 1 -> 0.0 0.0 1.0; limit lower=0.0 upper=0.13 effort=100 velocity=1.0 -> lower=0.0 upper=0.13 effort=100.0 velocity=1.0; origin xyz=0 0 0.013 rpy=2.91385731014123E-16 4.44300759504684E-17 3.25691080516352E-16 -> xyz=0.0 0.0 0.013 rpy=0.0 1.57655765344625e-30 -1.66533453693773e-16
- joint joint_arm_l3: axis 0 0 1 -> 0.0 0.0 1.0; limit lower=0.0 upper=0.13 effort=100 velocity=1.0 -> lower=0.0 upper=0.13 effort=100.0 velocity=1.0; origin xyz=0 0 0.013 rpy=3.5742E-16 3.2123E-16 -2.4565E-16 -> xyz=0.0 0.0 0.013 rpy=7.68831233799385e-30 2.36716479416092e-30 2.29652732251143e-17
- joint joint_arm_l4: axis 0 0 0 -> 0.0 0.0 0.0; origin xyz=-0.25471 0 0 rpy=1.5708 -3.1019E-16 -1.5708 -> xyz=-0.25900380552050645 -0.006563930614745515 0.005509129872430287 rpy=1.5889719525002595 -0.03244698018136405 -1.5686628459761205
- joint joint_aruco_inner_wrist: axis 0 0 0 -> 0.0 0.0 0.0; origin xyz=0.0472499999999947 -0.0119000000000034 -0.0272499999991938 rpy=3.14159265358979 4.23377442363088E-14 3.14159265358979 -> xyz=0.0472499999999947 -0.0119000000000034 -0.0272499999991938 rpy=3.14159265358979 4.23377442363088e-14 3.14159265358979
- joint joint_aruco_left_base: axis 0 0 0 -> 0.0 0.0 0.0; origin xyz=-0.00500000000000014 0.1304972 0.1597482 rpy=0 0 -1.5707963267949 -> xyz=-0.00500000000000014 0.1304972 0.1597482 rpy=0.0 0.0 -1.5707963267949
- joint joint_aruco_right_base: axis 0 0 0 -> 0.0 0.0 0.0; origin xyz=-0.00500000000000014 -0.1304972 0.1597482 rpy=0 0 -1.5707963267949 -> xyz=-0.0015028 -0.1304972 0.1597482 rpy=0.0 0.0 -1.5707963267949
- joint joint_aruco_shoulder: axis 0 0 0 -> 0.0 0.0 0.0; origin xyz=-0.0133768876375287 0.0558540528812078 0.0861368272417975 rpy=-1.53998860117704E-29 3.55962409571165E-15 0.0 -> xyz=-0.0133768876375287 0.0558540528812078 0.0861368272417975 rpy=-1.53998860117704e-29 3.55962409571165e-15 0.0
- joint joint_aruco_top_wrist: axis 0 0 0 -> 0.0 0.0 0.0; origin xyz=0.0472500000000019 0.0292850000000015 0 rpy=1.5707963267949 -8.03728587323464E-15 3.14159265358979 -> xyz=0.0472500000000019 0.0292850000000015 0.0 rpy=1.5707963267949 -8.03728587323464e-15 3.14159265358979
- joint joint_gripper_finger_left: axis 0 0 -1 -> 0.0 0.0 -1.0; limit lower=-0.6 upper=0.6 effort=100 velocity=1.0 -> lower=0.0 upper=0.0 effort=0.0 velocity=0.0; origin xyz=0.018599 0.003 0.033689 rpy=1.5708 -1.5708 0 -> xyz=0.0245029393015013 0.0 0.0371909405167127 rpy=-1.57079632679523 -1.48789318734672 -3.14159265358946; parent link_straight_gripper -> link_gripper_s3_body
- joint joint_gripper_finger_right: axis 0 0 1 -> 0.0 0.0 1.0; limit lower=-0.6 upper=0.6 effort=100 velocity=1.0 -> lower=0.0 upper=0.0 effort=0.0 velocity=0.0; origin xyz=-0.018599 0.003 0.033689 rpy=1.5708 1.5708 0 -> xyz=-0.0246929393014972 0.0 0.0371909405167257 rpy=-1.57079632679513 1.48789318732515 3.14159265358956; parent link_straight_gripper -> link_gripper_s3_body
- joint joint_gripper_fingertip_left: axis 0 0 0 -> 0.0 0.0 0.0; origin xyz=0.190596948563868 -0.015 0 rpy=1.57079632679496 4.51275387511463E-14 2.60113659715756 -> xyz=0.177784508377884 -0.0106721811879429 0.0 rpy=1.57079632679491 0.0 2.87979326579064
- joint joint_gripper_fingertip_right: axis 0 0 0 -> 0.0 0.0 0.0; origin xyz=-0.190596948563868 -0.015 0 rpy=-1.57079632679483 -3.43320051448326E-14 0.540456056432235 -> xyz=-0.177784508377902 -0.0106721811879468 0.0 rpy=-1.5707963267949 0.0 0.261799387799172
- joint joint_head: axis 0 0 0 -> 0.0 0.0 0.0; origin xyz=0 1.33 0 rpy=1.5708 -1.5615 3.1416 -> xyz=0.0 1.33 0.0 rpy=1.5707963267949 -1.5707963267949 3.1416
- joint joint_head_pan: axis 0 0 1 -> 0.0 0.0 1.0; limit lower=-3.9 upper=1.5 effort=100 velocity=1.0 -> lower=-3.9 upper=1.5 effort=100.0 velocity=1.0; origin xyz=0.135 0.0731 -0.003 rpy=-6.4986E-15 -6.068E-24 1.5708 -> xyz=0.1355499685444481 0.0773112249073356 0.0014758232430721568 rpy=0.0017186399547396195 0.00796009053320712 1.6094601685249763
- joint joint_head_tilt: axis 0 0 1 -> 0.0 0.0 1.0; limit lower=-1.53 upper=0.79 effort=100 velocity=1.0 -> lower=-1.53 upper=0.79 effort=100.0 velocity=1.0; origin xyz=-0.0013 0.027507 -0.053311 rpy=1.5708 6.068E-24 -2.5165E-15 -> xyz=0.0012654570348463422 0.027862124871306113 -0.04473556647529598 rpy=1.5786140964967674 0.0015421596711928665 0.027546588281587698
- joint joint_laser: axis 0 0 0 -> 0.0 0.0 0.0; origin xyz=0.000502800000000914 0 0.1664 rpy=0 0 -3.14159265358979 -> xyz=0.004 0.0 0.1664 rpy=0.0 0.0 3.1416
- joint joint_left_wheel: axis 0 0 1 -> 0.0 0.0 1.0; origin xyz=-0.00300000000001899 0.15765 0.0507999999999994 rpy=-1.5707963267949 3.16227047920818E-31 7.88745438253713E-16 -> xyz=0.0 0.17035 0.0508 rpy=-1.5708 2.6317e-16 -8.2057e-19
- joint joint_lift: axis 0 0 1 -> 0.0 0.0 1.0; limit lower=0.0 upper=1.1 effort=100 velocity=1.0 -> lower=0.0 upper=1.1 effort=100.0 velocity=1.0; origin xyz=-0.0369217062323472 0.165471199999996 -0.000341653286793524 rpy=-1.57079632679552 1.5615431375292 -6.2942004366467E-13 -> xyz=-0.037385 0.1666 0.0 rpy=-1.5708 1.5708 0.0
- joint joint_mast: axis 0 0 0 -> 0.0 0.0 0.0; origin xyz=-0.07 0.134999999999998 0.0284000000000001 rpy=1.5707963267949 0 0.00925318926571245 -> xyz=-0.07037253354767188 0.134819583812731 0.03779732532400868 rpy=1.5545415563018397 0.018375503066403454 -0.023961081343016256
- joint joint_respeaker: axis 0 0 0 -> 0.0 0.0 0.0; origin xyz=1.09074743137871E-05 1.36992 0.00303572796911382 rpy=1.57079632679553 0.0 3.14159265358916 -> xyz=0.0 1.37236408874452 0.00303065898329655 rpy=-1.5707963267949 -0.698131700797725 4.93295812652799e-16
- joint joint_right_wheel: axis 0 0 1 -> 0.0 0.0 1.0; origin xyz=-0.00300000000000034 -0.15765 0.0508000000000004 rpy=-1.57079632679489 -1.11022302462516E-16 7.28583859910277E-17 -> xyz=0.0 -0.17035 0.0508 rpy=-1.5708 1.2717e-16 4.8006e-17
- joint joint_wrist_pitch: axis 0 0 -1 -> 0.0 0.0 -1.0; limit lower=-1.57 upper=0.56 effort=100 velocity=1.0 -> lower=-1.57 upper=0.56 effort=100.0 velocity=1.0; origin xyz=0 -0.0195500000000002 -0.0247499999999984 rpy=1.5707963267949 -8.12895570882604E-15 -3.14159265358979 -> xyz=0.0 -0.019455 -0.0305 rpy=1.5708 0.0 3.1416
- joint joint_wrist_roll: axis 0 0 1 -> 0.0 0.0 1.0; limit lower=-3.14 upper=3.14 effort=100 velocity=1.0 -> lower=-3.14 upper=3.14 effort=100.0 velocity=1.0; origin xyz=-0.0188587444076125 -0.0239999999998942 0.01955 rpy=3.14159265358979 1.5707963267949 0 -> xyz=-0.018859 -0.024 0.01955 rpy=3.1416 1.5708 0.0
- joint joint_wrist_yaw: axis 0 0 -1 -> 0.0 0.0 -1.0; limit lower=-1.75 upper=4.0 effort=100 velocity=1.0 -> lower=-1.75 upper=4.0 effort=100.0 velocity=1.0; origin xyz=0.083 -0.03075 0 rpy=1.5708 4.2595E-14 2.6415E-15 -> xyz=0.0830000000000654 -0.0307500000000129 0.0 rpy=1.5708 4.2595e-14 2.6415e-15
- joint joint_wrist_yaw_bottom: axis 0 0 0 -> 0.0 0.0 0.0; origin xyz=0 0 0 rpy=-3.14159265358979 1.13367999021379E-14 1.57079632679489 -> xyz=0.0 0.0 0.0 rpy=-3.14159265358979 0.0 1.5707963267949
