Commit message: debugging

File: assets/hab_stretch/urdf/stretch_manip_mode.urdf (robot description, URDF)
Before this commit: robot stretch_description, 47 links, 46 joints
Links:
- added link fake_link_x, mass 0.749143203376
Joints:
- added joint joint_fake: type prismatic, parent base_link, child fake_link_x, origin xyz=0. 0. 0. rpy=0. 0. 0., axis 1.0 0.0 0.0, limit lower=-1.0 upper=1.1 effort=100.0 velocity=1.0
- joint joint_mast: parent base_link -> fake_link_x

Commit message: manipulation debug

File: assets/hab_stretch/urdf/stretch_manip_mode.urdf (robot description, URDF)
Before this commit: robot stretch_description, 48 links, 47 joints
Links:
- removed link base_theta_link
- removed link base_xy_link
- removed link world
- added link base_imu, mass 0.00092; collision mesh filename=package://stretch_description/meshes/base_imu.STL; visual mesh filename=package://stretch_description/meshes/base_imu.STL
- added link link_grasp_center
- link base_link: mass 1.1912 -> 17.384389; geometry collision mesh filename=package://stretch_description/meshes/base_link_collision.STL; visual mesh filename=package://stretch_description/meshes/base_link.STL
- link camera_link: geometry collision box size=0.02505 0.09 0.025; visual mesh filename=package://stretch_description/meshes/d435.dae
- link caster_link: geometry collision sphere radius=0.032; visual mesh filename=package://stretch_description/meshes/omni_wheel_m.STL
- link laser: mass 0.0749979022894495 -> 0.216007; geometry collision mesh filename=package://stretch_description/meshes/laser_collision.STL; visual mesh filename=package://stretch_description/meshes/laser.STL
- link link_arm_l0: mass 0.085003260946398 -> 0.427734; geometry collision mesh filename=package://stretch_description/meshes/link_arm_l0_collision.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; visual mesh filename=package://stretch_description/meshes/link_arm_l0.STL
- link link_arm_l1: mass 0.051382 -> 0.113658; geometry collision mesh filename=package://stretch_description/meshes/link_arm_l1_collision.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; visual mesh filename=package://stretch_description/meshes/link_arm_l1.STL
- link link_arm_l2: mass 0.0571386353275368 -> 0.130565; geometry collision mesh filename=package://stretch_description/meshes/link_arm_l2_collision.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; visual mesh filename=package://stretch_description/meshes/link_arm_l2.STL
- link link_arm_l3: mass 0.0628927381893134 -> 0.146817; geometry collision mesh filename=package://stretch_description/meshes/link_arm_l3_collision.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; visual mesh filename=package://stretch_description/meshes/link_arm_l3.STL
- link link_arm_l4: mass 0.068095 -> 0.235626; geometry collision mesh filename=package://stretch_description/meshes/link_arm_l4_collision.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; visual mesh filename=package://stretch_description/meshes/link_arm_l4.STL
- link link_aruco_inner_wrist: geometry collision mesh filename=package://stretch_description/meshes/link_aruco_inner_wrist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; visual mesh filename=package://stretch_description/meshes/link_aruco_inner_wrist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
- link link_aruco_left_base: geometry collision mesh filename=package://stretch_description/meshes/link_aruco_left_base.S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; visual mesh filename=package://stretch_description/meshes/link_aruco_left_base.S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
- link link_aruco_right_base: geometry collision mesh filename=package://stretch_description/meshes/link_aruco_right_base.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; visual mesh filename=package://stretch_description/meshes/link_aruco_right_base.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
- link link_aruco_shoulder: geometry collision mesh filename=package://stretch_description/meshes/link_aruco_shoulder.STL; visual mesh filename=package://stretch_description/meshes/link_aruco_shoulder.STL
- link link_aruco_top_wrist: geometry collision mesh filename=package://stretch_description/meshes/link_aruco_top_wrist.S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; visual mesh filename=package://stretch_description/meshes/link_aruco_top_wrist.S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
- link link_gripper_finger_left: mass 0.0476207785199479 -> 0.06; geometry collision mesh filename=package://stretch_description/meshes/link_gripper_finger_le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; visual mesh filename=package://stretch_description/meshes/link_gripper_finger_le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
- link link_gripper_finger_right: mass 0.047621 -> 0.06; geometry collision mesh filename=package://stretch_description/meshes/link_gripper_finger_ri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; visual mesh filename=package://stretch_description/meshes/link_gripper_finger_ri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
- link link_gripper_fingertip_left: mass 0.00382160686584851 -> 0.003822; geometry collision mesh filename=package://stretch_description/meshes/link_gripper_fingertip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; visual mesh filename=package://stretch_description/meshes/link_gripper_fingertip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
- link link_gripper_fingertip_right: mass 0.00382160881468841 -> 0.003822; geometry collision mesh filename=package://stretch_description/meshes/link_gripper_fingertip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; visual mesh filename=package://stretch_description/meshes/link_gripper_fingertip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
- link link_head: mass 0.133027236718691 -> 0.681871; geometry collision mesh filename=package://stretch_description/meshes/link_head_collision.STL; visual mesh filename=package://stretch_description/meshes/link_head.STL
- link link_head_pan: mass 0.0273764496535409 -> 0.062462; geometry collision mesh filename=package://stretch_description/meshes/link_head_pan_collisio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; visual mesh filename=package://stretch_description/meshes/link_head_pan.STL
- link link_head_tilt: mass 0.090217113313934 -> 0.283548; geometry collision mesh filename=package://stretch_description/meshes/link_head_tilt_collisi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; visual mesh filename=package://stretch_description/meshes/link_head_tilt.STL
- link link_left_wheel: mass 0.0042721 -> 0.20773; geometry collision mesh filename=package://stretch_description/meshes/link_left_wheel_collis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; visual mesh filename=package://stretch_description/meshes/link_left_wheel.STL
- link link_lift: mass 0.27218 -> 1.987167; geometry collision mesh filename=package://stretch_description/meshes/link_lift_collision.STL; visual mesh filename=package://stretch_description/meshes/link_lift.STL
- link link_mast: mass 1.8285 -> 1.764017; geometry collision mesh filename=package://stretch_description/meshes/link_mast_collision.STL; visual mesh filename=package://stretch_description/meshes/link_mast.STL
- link link_right_wheel: mass 0.0042721 -> 0.20773; geometry collision mesh filename=package://stretch_description/meshes/link_right_wheel_colli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; visual mesh filename=package://stretch_description/meshes/link_right_wheel.STL
- link link_straight_gripper: mass 0.0496384234458284 -> 0.147853; geometry collision mesh filename=package://stretch_description/meshes/link_straight_gripper_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; visual mesh filename=package://stretch_description/meshes/link_straight_gripper.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
- link link_wrist_pitch: mass 0.0701267146295583 -> 0.208129; geometry collision mesh filename=package://stretch_description/meshes/link_wrist_pitch_colli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; visual mesh filename=package://stretch_description/meshes/link_wrist_pitch.STL
- link link_wrist_roll: mass 0.00585666394358811 -> 0.01528; geometry collision mesh filename=package://stretch_description/meshes/link_wrist_roll_collis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; visual mesh filename=package://stretch_description/meshes/link_wrist_roll.STL
- link link_wrist_yaw: mass 0.0404746907425003 -> 0.054422; geometry collision mesh filename=package://stretch_description/meshes/link_wrist_yaw_collisi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; visual mesh filename=package://stretch_description/meshes/link_wrist_yaw.STL
- link link_wrist_yaw_bottom: mass 0.0988906816399982 -> 0.24284; geometry collision mesh filename=package://stretch_description/meshes/link_wrist_yaw_bottom_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; visual mesh filename=package://stretch_description/meshes/link_wrist_yaw_bottom.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
- link respeaker_base: mass 0.015643 -> 0.025175; geometry collision mesh filename=package://stretch_description/meshes/respeaker_base.STL; visual mesh filename=package://stretch_description/meshes/respeaker_base.STL
Joints:
- removed joint base_theta_joint
- removed joint base_x_joint
- removed joint base_y_joint
- added joint joint_base_imu: type fixed, parent base_link, child base_imu, origin xyz=-0.12838 0.0031592 0.1474 rpy=-3.1416 0.0 -1.5708, axis 0.0 0.0 0.0
- added joint joint_grasp_center: type fixed, parent link_straight_gripper, child link_grasp_center, origin xyz=0.0 0.0 0.23 rpy=-1.5707963267949 -1.5707963267949 0.0
- joint camera_joint: origin xyz=0.02802960503838624 -0.007608222297947431 0.018218494141479257 rpy=0.010658876360659654 -0.0022761048951753793 0.018675317090921212 -> xyz=0.025280607108926732 -0.013667484906757996 0.017739850624818598 rpy=-0.0009652884720215551 0.023054303721607772 0.03853450363377455
- joint joint_arm_l4: origin xyz=-0.25956015433181046 -0.0059261537843136765 -0.005557384627505743 rpy=1.5619286973774569 -0.006924580188019336 -1.575847166561953 -> xyz=-0.26071485771276837 -0.0015985411337465219 -0.0017742513625829514 rpy=1.586071184113442 0.006734738344140068 -1.5516013728847526
- joint joint_head_pan: origin xyz=0.1284513021260868 0.07637128403435504 0.00023722543808071166 rpy=-0.013467967166369273 0.005690738105448956 1.6024957766579377 -> xyz=0.13946205358565067 0.0715510730766181 0.002433848249537541 rpy=0.007858631731799605 0.007772825286872953 1.5402416889676325
- joint joint_head_tilt: origin xyz=0.0032337815907659225 0.030910701770693223 -0.04783143162927699 rpy=1.5763332066189244 -0.029319157204454882 -0.005080558641851002 -> xyz=0.001983888991630815 0.022254345636052615 -0.060227066766224406 rpy=1.544503242574277 -0.007932491465490576 -0.04876088906076381
- joint joint_mast: origin xyz=-0.07174416574437388 0.13780491000396983 0.03663931715774088 rpy=1.5780076046568878 0.016499709009588637 -0.007971437955302632 -> xyz=-0.06671430129673842 0.14027841219737333 0.033867009722517646 rpy=1.5769186882626829 -0.022012875790222264 0.006707186804730073

Commit message: update

File: assets/hab_stretch/urdf/stretch_manip_mode.urdf (robot description, URDF)
Before this commit: robot stretch, 47 links, 46 joints
Links:
- removed link link_straight_gripper
- added link link_aruco_d405, mass 0.000393662237156561; collision mesh filename=package://stretch_description/meshes/link_SG3_aruco_d405.STL; visual mesh filename=package://stretch_description/meshes/link_SG3_aruco_d405.STL
- added link link_aruco_fingertip_left, mass 7.44175884388882e-05; collision mesh filename=package://stretch_description/meshes/link_SG3_aruco_fingert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; visual mesh filename=package://stretch_description/meshes/link_SG3_aruco_fingert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
- added link link_aruco_fingertip_right, mass 7.44175884388862e-05; collision mesh filename=package://stretch_description/meshes/link_SG3_aruco_fingert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; visual mesh filename=package://stretch_description/meshes/link_SG3_aruco_fingert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
- added link link_gripper_s3_body, mass 0.288995995074102; collision mesh filename=package://stretch_description/meshes/link_SG3_gripper_body_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; visual mesh filename=package://stretch_description/meshes/link_SG3_gripper_body.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
- added link link_head_nav_cam, mass 0.028346169831483; collision mesh filename=package://stretch_description/meshes/link_SE3_head_nav_cam_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; visual mesh filename=package://stretch_description/meshes/link_SE3_head_nav_cam.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
- added link link_wrist_quick_connect
- link link_gripper_finger_left: mass 0.06 -> 0.0483698266031602; geometry collision mesh filename=package://stretch_description/meshes/link_SG3_gripper_finge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; visual mesh filename=package://stretch_description/meshes/link_SG3_gripper_finge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
- link link_gripper_finger_right: mass 0.06 -> 0.0483698337858479; geometry collision mesh filename=package://stretch_description/meshes/link_SG3_gripper_finge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; visual mesh filename=package://stretch_description/meshes/link_SG3_gripper_finge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
- link link_gripper_fingertip_left: mass 0.003822 -> 0.00382162054362131; geometry collision mesh filename=package://stretch_description/meshes/link_SG3_gripper_finge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; visual mesh filename=package://stretch_description/meshes/link_SG3_gripper_finge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
- link link_gripper_fingertip_right: mass 0.003822 -> 0.00382162062525088; geometry collision mesh filename=package://stretch_description/meshes/link_SG3_gripper_finge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; visual mesh filename=package://stretch_description/meshes/link_SG3_gripper_finge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
- link link_wrist_pitch: mass 0.208129 -> 0.116590512374845; geometry collision mesh filename=package://stretch_description/meshes/link_DW3_wrist_pitch_c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; visual mesh filename=package://stretch_description/meshes/link_DW3_wrist_pitch.S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
- link link_wrist_roll: mass 0.01528 -> 0.0221916689638078; geometry collision mesh filename=package://stretch_description/meshes/link_DW3_wrist_roll_co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; visual mesh filename=package://stretch_description/meshes/link_DW3_wrist_roll.STL
- link link_wrist_yaw_bottom: mass 0.24284 -> 0.144548635554334; geometry collision mesh filename=package://stretch_description/meshes/link_DW3_wrist_yaw_bot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; visual mesh filename=package://stretch_description/meshes/link_DW3_wrist_yaw_bot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
Joints:
- removed joint joint_straight_gripper
- added joint joint_aruco_d405: type fixed, parent link_gripper_s3_body, child link_aruco_d405, origin xyz=0.0 0.0671264013906604 0.0297716109784749 rpy=2.96705999342568 -0.000305721573415565 3.1398588194619, axis 0.0 0.0 0.0
- added joint joint_aruco_fingertip_left: type fixed, parent link_gripper_finger_left, child link_aruco_fingertip_left, origin xyz=0.143934974292929 -0.00436381846064454 -8.58640479230455e-05 rpy=-1.76278254451424 0.0 0.959931088596885, axis 0.0 0.0 0.0
- added joint joint_aruco_fingertip_right: type fixed, parent link_gripper_finger_right, child link_aruco_fingertip_right, origin xyz=-0.143934974292953 -0.00436381846065068 -8.58640479174944e-05 rpy=-1.76278254451426 0.0 -0.959931088596862, axis 0.0 0.0 0.0
- added joint joint_gripper_s3_body: type fixed, parent link_wrist_roll, child link_gripper_s3_body, origin xyz=0.0 0.0 0.0209999999993159 rpy=0.0 0.0 -3.14159265358975, axis 0.0 0.0 0.0
- added joint joint_head_nav_cam: type fixed, parent link_head_tilt, child link_head_nav_cam, origin xyz=0.0402000000000069 -0.0411729746231231 -0.0245785717313561 rpy=0.0 1.5707963267949 0.0, axis 0.0 0.0 0.0
- added joint joint_wrist_quick_connect: type fixed, parent link_wrist_roll, child link_wrist_quick_connect, origin xyz=0.0 0.0 0.0085 rpy=1.5708 0.0 -1.5708, axis 0.0 0.0 0.0
- joint camera_joint: origin xyz=0.025280607108926732 -0.013667484906757996 0.017739850624818598 rpy=-0.0009652884720215551 0.023054303721607772 0.03853450363377455 -> xyz=0.027491210169072782 -0.008099935183508883 0.017006240598738752 rpy=0.007046694733527481 0.0036560752538217223 -0.03688734326513847
- joint joint_arm_l4: origin xyz=-0.26071485771276837 -0.0015985411337465219 -0.0017742513625829514 rpy=1.586071184113442 0.006734738344140068 -1.5516013728847526 -> xyz=-0.2608650244668732 0.0029169778606417548 0.0017127107828243482 rpy=1.5733190166907038 0.042439274543223604 -1.5808019766990344
- joint joint_grasp_center: origin xyz=0.0 0.0 0.23 rpy=-1.5707963267949 -1.5707963267949 0.0 -> xyz=0.0 0.0 0.23 rpy=-1.5707963267949 -1.5707963267948 0.0; parent link_straight_gripper -> link_gripper_s3_body
- joint joint_gripper_finger_left: limit lower=-0.6 upper=0.6 effort=100.0 velocity=1.0 -> lower=0.0 upper=0.0 effort=0.0 velocity=0.0; origin xyz=0.018599 0.003 0.033689 rpy=1.5708 -1.5708 0.0 -> xyz=0.0245029393015013 0.0 0.0371909405167127 rpy=-1.57079632679523 -1.48789318734672 -3.14159265358946; parent link_straight_gripper -> link_gripper_s3_body
- joint joint_gripper_finger_right: limit lower=-0.6 upper=0.6 effort=100.0 velocity=1.0 -> lower=0.0 upper=0.0 effort=0.0 velocity=0.0; origin xyz=-0.018599 0.003 0.033689 rpy=1.5708 1.5708 0.0 -> xyz=-0.0246929393014972 0.0 0.0371909405167257 rpy=-1.57079632679513 1.48789318732515 3.14159265358956; parent link_straight_gripper -> link_gripper_s3_body
- joint joint_gripper_fingertip_left: origin xyz=0.190596948563868 -0.015 0.0 rpy=1.57079632679496 4.51275387511463e-14 2.60113659715756 -> xyz=0.177784508377884 -0.0106721811879429 0.0 rpy=1.57079632679491 0.0 2.87979326579064
- joint joint_gripper_fingertip_right: origin xyz=-0.190596948563868 -0.015 0.0 rpy=-1.57079632679483 -3.43320051448326e-14 0.540456056432235 -> xyz=-0.177784508377902 -0.0106721811879468 0.0 rpy=-1.5707963267949 0.0 0.261799387799172
- joint joint_head_pan: origin xyz=0.13946205358565067 0.0715510730766181 0.002433848249537541 rpy=0.007858631731799605 0.007772825286872953 1.5402416889676325 -> xyz=0.138528977923653 0.07499632874010914 0.0030468218584924173 rpy=3.2485935060467686e-05 0.00893058065850405 1.6542704589420498
- joint joint_head_tilt: origin xyz=0.001983888991630815 0.022254345636052615 -0.060227066766224406 rpy=1.544503242574277 -0.007932491465490576 -0.04876088906076381 -> xyz=0.001107931486650946 0.023720056316094976 -0.04936267653073215 rpy=1.5790860939266764 -0.0805411511581009 0.022950759695878096
- joint joint_mast: origin xyz=-0.06671430129673842 0.14027841219737333 0.033867009722517646 rpy=1.5769186882626829 -0.022012875790222264 0.006707186804730073 -> xyz=-0.06883017193407229 0.13630384540724177 0.03810045295473849 rpy=1.5502932034054995 -0.031218646376585557 0.01925607057301884
- joint joint_wrist_pitch: origin xyz=0.0 -0.0195500000000002 -0.0247499999999984 rpy=1.5707963267949 -8.12895570882604e-15 -3.14159265358979 -> xyz=0.0 -0.019455 -0.0305 rpy=1.5708 0.0 3.1416
- joint joint_wrist_roll: origin xyz=-0.0188587444076125 -0.0239999999998942 0.01955 rpy=3.14159265358979 1.5707963267949 0.0 -> xyz=-0.018859 -0.024 0.01955 rpy=3.1416 1.5708 0.0
- joint joint_wrist_yaw_bottom: origin xyz=0.0 0.0 0.0 rpy=-3.14159265358979 1.13367999021379e-14 1.57079632679489 -> xyz=0.0 0.0 0.0 rpy=-3.14159265358979 0.0 1.5707963267949
