Commit message: update

File: assets/hab_stretch/urdf/stretch_manip_mode.urdf (robot description, URDF)
Before this commit: robot stretch, 52 links, 51 joints
Links:
- removed link link_aruco_d405
- removed link link_aruco_fingertip_left
- removed link link_aruco_fingertip_right
- removed link link_gripper_s3_body
- removed link link_head_nav_cam
- removed link link_wrist_quick_connect
- added link link_straight_gripper, mass 0.147853; collision mesh filename=package://stretch_description/meshes/link_straight_gripper_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; visual mesh filename=package://stretch_description/meshes/link_straight_gripper.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
- link link_gripper_finger_left: mass 0.0483698266031602 -> 0.06; geometry collision mesh filename=package://stretch_description/meshes/link_gripper_finger_le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; visual mesh filename=package://stretch_description/meshes/link_gripper_finger_le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
- link link_gripper_finger_right: mass 0.0483698337858479 -> 0.06; geometry collision mesh filename=package://stretch_description/meshes/link_gripper_finger_ri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; visual mesh filename=package://stretch_description/meshes/link_gripper_finger_ri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
- link link_gripper_fingertip_left: mass 0.00382162054362131 -> 0.003822; geometry collision mesh filename=package://stretch_description/meshes/link_gripper_fingertip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; visual mesh filename=package://stretch_description/meshes/link_gripper_fingertip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
- link link_gripper_fingertip_right: mass 0.00382162062525088 -> 0.003822; geometry collision mesh filename=package://stretch_description/meshes/link_gripper_fingertip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; visual mesh filename=package://stretch_description/meshes/link_gripper_fingertip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
- link link_wrist_pitch: mass 0.116590512374845 -> 0.208129; geometry collision mesh filename=package://stretch_description/meshes/link_wrist_pitch_colli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; visual mesh filename=package://stretch_description/meshes/link_wrist_pitch.STL
- link link_wrist_roll: mass 0.0221916689638078 -> 0.01528; geometry collision mesh filename=package://stretch_description/meshes/link_wrist_roll_collis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; visual mesh filename=package://stretch_description/meshes/link_wrist_roll.STL
- link link_wrist_yaw_bottom: mass 0.144548635554334 -> 0.24284; geometry collision mesh filename=package://stretch_description/meshes/link_wrist_yaw_bottom_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; visual mesh filename=package://stretch_description/meshes/link_wrist_yaw_bottom.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
Joints:
- removed joint joint_aruco_d405
- removed joint joint_aruco_fingertip_left
- removed joint joint_aruco_fingertip_right
- removed joint joint_gripper_s3_body
- removed joint joint_head_nav_cam
- removed joint joint_wrist_quick_connect
- added joint joint_straight_gripper: type fixed, parent link_wrist_roll, child link_straight_gripper, origin xyz=0.0 0.0 0.0155 rpy=3.54987407349455e-30 3.24021254484265e-20 -3.14159265358979, axis 0.0 0.0 0.0
- joint camera_joint: origin xyz=0.027491210169072782 -0.008099935183508883 0.017006240598738752 rpy=0.007046694733527481 0.0036560752538217223 -0.03688734326513847 -> xyz=0.027848092689966176 -0.008192081891921481 0.019699144735927685 rpy=0.0020850946809237905 -0.016175552135467397 0.0069624349423955505
- joint joint_arm_l4: origin xyz=-0.2608650244668732 0.0029169778606417548 0.0017127107828243482 rpy=1.5733190166907038 0.042439274543223604 -1.5808019766990344 -> xyz=-0.2554280576880445 -0.0034267659889070197 0.009297206693180219 rpy=1.5762403594474133 -0.032942947075947915 -1.5950145467759027
- joint joint_grasp_center: origin xyz=0.0 0.0 0.23 rpy=-1.5707963267949 -1.5707963267948 0.0 -> xyz=0.0 0.0 0.23 rpy=-1.5707963267949 -1.5707963267949 0.0; parent link_gripper_s3_body -> link_straight_gripper
- joint joint_gripper_finger_left: limit lower=0.0 upper=0.0 effort=0.0 velocity=0.0 -> lower=-0.6 upper=0.6 effort=100.0 velocity=1.0; origin xyz=0.0245029393015013 0.0 0.0371909405167127 rpy=-1.57079632679523 -1.48789318734672 -3.14159265358946 -> xyz=0.018599 0.003 0.033689 rpy=1.5708 -1.5708 0.0; parent link_gripper_s3_body -> link_straight_gripper
- joint joint_gripper_finger_right: limit lower=0.0 upper=0.0 effort=0.0 velocity=0.0 -> lower=-0.6 upper=0.6 effort=100.0 velocity=1.0; origin xyz=-0.0246929393014972 0.0 0.0371909405167257 rpy=-1.57079632679513 1.48789318732515 3.14159265358956 -> xyz=-0.018599 0.003 0.033689 rpy=1.5708 1.5708 0.0; parent link_gripper_s3_body -> link_straight_gripper
- joint joint_gripper_fingertip_left: origin xyz=0.177784508377884 -0.0106721811879429 0.0 rpy=1.57079632679491 0.0 2.87979326579064 -> xyz=0.190596948563868 -0.015 0.0 rpy=1.57079632679496 4.51275387511463e-14 2.60113659715756
- joint joint_gripper_fingertip_right: origin xyz=-0.177784508377902 -0.0106721811879468 0.0 rpy=-1.5707963267949 0.0 0.261799387799172 -> xyz=-0.190596948563868 -0.015 0.0 rpy=-1.57079632679483 -3.43320051448326e-14 0.540456056432235
- joint joint_head_pan: origin xyz=0.138528977923653 0.07499632874010914 0.0030468218584924173 rpy=3.2485935060467686e-05 0.00893058065850405 1.6542704589420498 -> xyz=0.13550459909834245 0.07449577337076961 0.006355639835664768 rpy=-0.0007308145293812751 0.007705460698482991 1.5773575464502596
- joint joint_head_tilt: origin xyz=0.001107931486650946 0.023720056316094976 -0.04936267653073215 rpy=1.5790860939266764 -0.0805411511581009 0.022950759695878096 -> xyz=0.003101639774150571 0.0323182686288255 -0.048010625693505 rpy=1.5922076083155883 -0.024161969233451375 0.0804552813326012
- joint joint_mast: origin xyz=-0.06883017193407229 0.13630384540724177 0.03810045295473849 rpy=1.5502932034054995 -0.031218646376585557 0.01925607057301884 -> xyz=-0.07066491395701623 0.1366433023962791 0.037547096703931755 rpy=1.5690789216589467 -0.007235921898443909 0.014953116910468222
- joint joint_wrist_pitch: origin xyz=0.0 -0.019455 -0.0305 rpy=1.5708 0.0 3.1416 -> xyz=0.0 -0.0195500000000002 -0.0247499999999984 rpy=1.5707963267949 -8.12895570882604e-15 -3.14159265358979
- joint joint_wrist_roll: origin xyz=-0.018859 -0.024 0.01955 rpy=3.1416 1.5708 0.0 -> xyz=-0.0188587444076125 -0.0239999999998942 0.01955 rpy=3.14159265358979 1.5707963267949 0.0
- joint joint_wrist_yaw_bottom: origin xyz=0.0 0.0 0.0 rpy=-3.14159265358979 0.0 1.5707963267949 -> xyz=0.0 0.0 0.0 rpy=-3.14159265358979 1.13367999021379e-14 1.57079632679489

Commit message: update

File: assets/hab_stretch/urdf/stretch_manip_mode.urdf (robot description, URDF)
Before this commit: robot stretch_description, 47 links, 46 joints
Joints:
- joint camera_joint: origin xyz=0.027848092689966176 -0.008192081891921481 0.019699144735927685 rpy=0.0020850946809237905 -0.016175552135467397 0.0069624349423955505 -> xyz=0.02638119730898156 -0.008992984306469253 0.019035293929558446 rpy=0.003918821957098094 0.008027010997255335 0.02118662837117397
- joint joint_arm_l4: origin xyz=-0.2554280576880445 -0.0034267659889070197 0.009297206693180219 rpy=1.5762403594474133 -0.032942947075947915 -1.5950145467759027 -> xyz=-0.2597108931717514 -0.0017208937614510268 0.005240546783706932 rpy=1.574015041340944 -0.02552587253464722 -1.5797054921069134
- joint joint_head_pan: origin xyz=0.13550459909834245 0.07449577337076961 0.006355639835664768 rpy=-0.0007308145293812751 0.007705460698482991 1.5773575464502596 -> xyz=0.13901387823584807 0.07162424327732812 0.0022155565040961407 rpy=0.0020073855055640563 0.003210717055941892 1.6566090911876217
- joint joint_head_tilt: origin xyz=0.003101639774150571 0.0323182686288255 -0.048010625693505 rpy=1.5922076083155883 -0.024161969233451375 0.0804552813326012 -> xyz=0.00318539759013445 0.029109131406915165 -0.04563278282593967 rpy=1.5715479580303684 0.04155459084730628 -0.0011455505917390039
- joint joint_mast: origin xyz=-0.07066491395701623 0.1366433023962791 0.037547096703931755 rpy=1.5690789216589467 -0.007235921898443909 0.014953116910468222 -> xyz=-0.0703318702765198 0.13532611168442982 0.037730738458300474 rpy=1.5450345873026095 -0.031182340346273207 0.015146911467056615

Commit message: update

File: assets/hab_stretch/urdf/stretch_manip_mode.urdf (robot description, URDF)
Before this commit: robot stretch_description, 47 links, 46 joints
Joints:
- joint camera_joint: origin xyz=0.02638119730898156 -0.008992984306469253 0.019035293929558446 rpy=0.003918821957098094 0.008027010997255335 0.02118662837117397 -> xyz=0.025592555468793427 -0.01449736657070223 0.01872009176926669 rpy=-0.009100463976788549 0.01911053783740657 0.03649843715753866
- joint joint_arm_l4: origin xyz=-0.2597108931717514 -0.0017208937614510268 0.005240546783706932 rpy=1.574015041340944 -0.02552587253464722 -1.5797054921069134 -> xyz=-0.25986890556581715 0.0008644329707763534 -0.005043672476175837 rpy=1.5920025388009347 -0.017416365130188183 -1.5733393262116346
- joint joint_head_pan: origin xyz=0.13901387823584807 0.07162424327732812 0.0022155565040961407 rpy=0.0020073855055640563 0.003210717055941892 1.6566090911876217 -> xyz=0.14285342465715847 0.07184125289972697 0.002214091867859479 rpy=0.004742924965478492 0.021979321375489302 1.6034244978598249
- joint joint_head_tilt: origin xyz=0.00318539759013445 0.029109131406915165 -0.04563278282593967 rpy=1.5715479580303684 0.04155459084730628 -0.0011455505917390039 -> xyz=-6.743437609460197e-06 0.02558491440903574 -0.0596432581666555 rpy=1.5597629576003158 -0.044884516136375785 0.06227598589278792
- joint joint_mast: origin xyz=-0.0703318702765198 0.13532611168442982 0.037730738458300474 rpy=1.5450345873026095 -0.031182340346273207 0.015146911467056615 -> xyz=-0.06889459118401083 0.13801249646288638 0.03603096916165477 rpy=1.577273841344249 -0.020438660992705637 0.03582731011578926

Commit message: update

File: assets/hab_stretch/urdf/stretch_manip_mode.urdf (robot description, URDF)
Before this commit: robot stretch, 47 links, 46 joints
Joints:
- joint camera_joint: origin xyz=0.025592555468793427 -0.01449736657070223 0.01872009176926669 rpy=-0.009100463976788549 0.01911053783740657 0.03649843715753866 -> xyz=0.02638119730898156 -0.008992984306469253 0.019035293929558446 rpy=0.003918821957098094 0.008027010997255335 0.02118662837117397
- joint joint_arm_l4: origin xyz=-0.25986890556581715 0.0008644329707763534 -0.005043672476175837 rpy=1.5920025388009347 -0.017416365130188183 -1.5733393262116346 -> xyz=-0.2597108931717514 -0.0017208937614510268 0.005240546783706932 rpy=1.574015041340944 -0.02552587253464722 -1.5797054921069134
- joint joint_head_pan: origin xyz=0.14285342465715847 0.07184125289972697 0.002214091867859479 rpy=0.004742924965478492 0.021979321375489302 1.6034244978598249 -> xyz=0.13901387823584807 0.07162424327732812 0.0022155565040961407 rpy=0.0020073855055640563 0.003210717055941892 1.6566090911876217
- joint joint_head_tilt: origin xyz=-6.743437609460197e-06 0.02558491440903574 -0.0596432581666555 rpy=1.5597629576003158 -0.044884516136375785 0.06227598589278792 -> xyz=0.00318539759013445 0.029109131406915165 -0.04563278282593967 rpy=1.5715479580303684 0.04155459084730628 -0.0011455505917390039
- joint joint_mast: origin xyz=-0.06889459118401083 0.13801249646288638 0.03603096916165477 rpy=1.577273841344249 -0.020438660992705637 0.03582731011578926 -> xyz=-0.0703318702765198 0.13532611168442982 0.037730738458300474 rpy=1.5450345873026095 -0.031182340346273207 0.015146911467056615
